Commit message: Update wheel dimensions and inertia values

File: urdf/barista_robot_model.urdf (robot description, URDF)
Before this commit: robot barista_robot, 14 links, 13 joints
Links:
- link caster_wheel_pitch_link: mass 0.010 -> 0.030; geometry collision sphere radius=0.0176; visual sphere radius=0.0176
- link left_wheel_link: geometry collision cylinder length=0.0206 radius=0.0352; visual cylinder length=0.0206 radius=0.0352
- link right_wheel_link: geometry collision cylinder length=0.0178 radius=0.0352; visual cylinder length=0.0206 radius=0.0352
Joints:
- joint bottom_joint: origin xyz=0 0 0.094 rpy=0 0 0 -> xyz=0 0 0.0951 rpy=0 0 0
- joint left_wheel_joint: origin xyz=0 0.158 -0.061 rpy=0 1.571 1.571 -> xyz=0 0.158 -0.0599 rpy=0 1.571 1.571
- joint right_wheel_joint: origin xyz=0 -0.158 -0.061 rpy=0 1.571 1.571 -> xyz=0 -0.158 -0.0599 rpy=0 1.571 1.571

Commit message: Joint states publisher not working

File: urdf/barista_robot_model.urdf (robot description, URDF)
Before this commit: robot barista_robot, 14 links, 13 joints
Links:
- removed link bottom_link
- removed link caster_wheel_pitch_link
- removed link caster_wheel_roll_link
- removed link caster_wheel_yaw_link
- removed link spacer_1_link
- removed link spacer_2_link
- removed link spacer_3_link
- removed link spacer_4_link
- removed link top_link
- added link back_caster_wheel_pitch_link, mass 0.030; collision sphere radius=0.0176; visual sphere radius=0.0176
- added link back_caster_wheel_roll_link, mass 0.001; collision cylinder length=0.001 radius=0.0045000000000000005; visual cylinder length=0.001 radius=0.0045000000000000005
- added link back_caster_wheel_yaw_link, mass 0.001; collision cylinder length=0.001 radius=0.0045000000000000005; visual cylinder length=0.001 radius=0.0045000000000000005
- added link body_link, mass 0.100; collision cylinder length=0.155 radius=0.178; visual cylinder length=0.155 radius=0.178
- added link cup_holder_tray_link, mass 0.050; collision cylinder length=0.090 radius=0.160; visual cylinder length=0.090 radius=0.160
- added link front_caster_wheel_pitch_link, mass 0.030; collision sphere radius=0.0176; visual sphere radius=0.0176
- added link front_caster_wheel_roll_link, mass 0.001; collision cylinder length=0.001 radius=0.0045000000000000005; visual cylinder length=0.001 radius=0.0045000000000000005
- added link front_caster_wheel_yaw_link, mass 0.001; collision cylinder length=0.001 radius=0.0045000000000000005; visual cylinder length=0.001 radius=0.0045000000000000005
- added link standoff_rod_1_link, mass 0.020; collision cylinder length=0.220 radius=0.010; visual cylinder length=0.220 radius=0.010
- added link standoff_rod_2_link, mass 0.020; collision cylinder length=0.220 radius=0.010; visual cylinder length=0.220 radius=0.010
- added link standoff_rod_3_link, mass 0.020; collision cylinder length=0.220 radius=0.010; visual cylinder length=0.220 radius=0.010
- added link standoff_rod_4_link, mass 0.020; collision cylinder length=0.220 radius=0.010; visual cylinder length=0.220 radius=0.010
Joints:
- removed joint bottom_joint
- removed joint caster_wheel_pitch_joint
- removed joint caster_wheel_roll_joint
- removed joint caster_wheel_yaw_joint
- removed joint spacer_1_joint
- removed joint spacer_2_joint
- removed joint spacer_3_joint
- removed joint spacer_4_joint
- removed joint top_joint
- added joint back_caster_wheel_pitch_joint: type continuous, parent back_caster_wheel_roll_link, child back_caster_wheel_pitch_link, origin xyz=0 0 0 rpy=0 0 0, axis 0 1 0, limit effort=1000.0 velocity=100.0
- added joint back_caster_wheel_roll_joint: type continuous, parent back_caster_wheel_yaw_link, child back_caster_wheel_roll_link, origin xyz=0 0 0 rpy=0 0 0, axis 1 0 0, limit effort=1000.0 velocity=100.0
- added joint back_caster_wheel_yaw_joint: type continuous, parent body_link, child back_caster_wheel_yaw_link, origin xyz=-0.158 0 -0.0775 rpy=0 0 0, axis 0 0 1, limit effort=1000.0 velocity=100.0
- added joint body_joint: type fixed, parent base_link, child body_link, origin xyz=0 0 0.0951 rpy=0 0 0
- added joint cup_holder_tray_joint: type fixed, parent body_link, child cup_holder_tray_link, origin xyz=0 0 0.3425 rpy=0 0 0
- added joint front_caster_wheel_pitch_joint: type continuous, parent front_caster_wheel_roll_link, child front_caster_wheel_pitch_link, origin xyz=0 0 0 rpy=0 0 0, axis 0 1 0, limit effort=1000.0 velocity=100.0
- added joint front_caster_wheel_roll_joint: type continuous, parent front_caster_wheel_yaw_link, child front_caster_wheel_roll_link, origin xyz=0 0 0 rpy=0 0 0, axis 1 0 0, limit effort=1000.0 velocity=100.0
- added joint front_caster_wheel_yaw_joint: type continuous, parent body_link, child front_caster_wheel_yaw_link, origin xyz=0.158 0 -0.0775 rpy=0 0 0, axis 0 0 1, limit effort=1000.0 velocity=100.0
- added joint standoff_rod_1_link_joint: type fixed, parent body_link, child standoff_rod_1_link, origin xyz=-0.030 -0.128 0.1875 rpy=0 0 0
- added joint standoff_rod_2_joint: type fixed, parent body_link, child standoff_rod_2_link, origin xyz=-0.030 0.128 0.1875 rpy=0 0 0
- added joint standoff_rod_3_joint: type fixed, parent body_link, child standoff_rod_3_link, origin xyz=0.030 -0.128 0.1875 rpy=0 0 0
- added joint standoff_rod_4_joint: type fixed, parent body_link, child standoff_rod_4_link, origin xyz=0.030 0.128 0.1875 rpy=0 0 0
- joint left_wheel_joint: parent bottom_link -> body_link
- joint lidar_support_joint: parent bottom_link -> body_link
- joint right_wheel_joint: parent bottom_link -> body_link

Commit message: Add lidar mesh and gazebo world, improve launch file and urdf description

File: urdf/barista_robot_model.urdf (robot description, URDF)
Before this commit: robot barista_robot, 17 links, 16 joints
Links:
- removed link lidar_spinner_link
- removed link lidar_support_link
- added link lidar_link, mass 0.050; collision mesh filename=package://barista_robot_description/meshes/hokuyo_urg_04lx.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 scale=1 1 1; visual mesh filename=package://barista_robot_description/meshes/hokuyo_urg_04lx.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 scale=1 1 1
Joints:
- removed joint lidar_spinner_joint
- removed joint lidar_support_joint
- added joint lidar_joint: type fixed, parent body_link, child lidar_link, origin xyz=0.100 0 0.0775 rpy=0 0 0

Commit message: Include conditional for laser scanner, unified rviz config and laser scanner name

File: urdf/barista_robot_model.urdf (robot description, URDF)
Before this commit: robot barista_robot, 16 links, 15 joints
Links:
- removed link lidar_link
- added link laser_scanner_link, mass 0.050; collision mesh filename=package://barista_robot_description/meshes/hokuyo_urg_04lx.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 scale=1 1 1; visual mesh filename=package://barista_robot_description/meshes/hokuyo_urg_04lx.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 scale=1 1 1
Joints:
- removed joint lidar_joint
- added joint laser_scanner_joint: type fixed, parent body_link, child laser_scanner_link, origin xyz=0.100 0 0.0775 rpy=0 0 0

File: xacro/barista_robot_model.urdf.xacro (robot description, xacro)
@@ -1,4 +1,6 @@
 <?xml version="1.0"?>
 <robot xmlns:xacro="http://www.ros.org/wiki/xacro" name="barista_robot">
+<xacro:property name="include_laser" value="$(arg include_laser)"/>
+<xacro:arg name="include_laser" default="true"/>
 <xacro:include filename="$(find barista_robot_description)/xacro/caster_wheel.xacro" />
 <xacro:include filename="$(find barista_robot_description)/xacro/cup_holder_tray.xacro" />
@@ -18,8 +20,10 @@
 <xacro:standoff_rod standoff_rod_name="standoff_rod_4"/>
 <xacro:cup_holder_tray/>
-<xacro:laser_scanner/>
+<xacro:if value="${include_laser}">
+  <xacro:laser_scanner/>
+  <xacro:laser_scanner_plugin/>
+</xacro:if>
 <xacro:state_publisher/>
 <xacro:differential_drive/>
-<xacro:laser_scanner_plugin/>
 <xacro:rviz_materials/>
 <xacro:gazebo_elements/>
@@ -143,8 +147,10 @@
   </joint>
   <!-- Lidar -->
-  <joint name="laser_scanner_joint" type="fixed">
-    <origin rpy="0 0 0" xyz="0.100 0 0.0775"/>
-    <parent link="body_link"/>
-    <child link="laser_scanner_link"/>
-  </joint>
+  <xacro:if value="${include_laser}">
+    <joint name="laser_scanner_joint" type="fixed">
+      <origin rpy="0 0 0" xyz="0.100 0 0.0775"/>
+      <parent link="body_link"/>
+      <child link="laser_scanner_link"/>
+    </joint>
+  </xacro:if>
 </robot>

Commit message: Update wheel location

File: urdf/barista_robot_model.urdf (robot description, URDF)
Before this commit: robot barista_robot, 16 links, 15 joints
Joints:
- joint back_caster_wheel_yaw_joint: origin xyz=-0.158 0 -0.0775 rpy=0 0 0 -> xyz=-0.140 0 -0.0775 rpy=0 0 0
- joint front_caster_wheel_yaw_joint: origin xyz=0.158 0 -0.0775 rpy=0 0 0 -> xyz=0.140 0 -0.0775 rpy=0 0 0
- joint left_wheel_joint: origin xyz=0 0.158 -0.0599 rpy=0 1.571 1.571 -> xyz=0 0.140 -0.0599 rpy=0 1.571 1.571
- joint right_wheel_joint: origin xyz=0 -0.158 -0.0599 rpy=0 1.571 1.571 -> xyz=0 -0.140 -0.0599 rpy=0 1.571 1.571

File: xacro/barista_robot_model.urdf.xacro (robot description, xacro)
@@ -76,5 +76,5 @@
   <!-- Wheels joint -->
   <joint name="left_drive_wheel_joint" type="continuous">
-    <origin rpy="0 1.571 1.571" xyz="0 0.158 -0.0599"/>
+    <origin rpy="0 1.571 1.571" xyz="0 0.140 -0.0599"/>
     <parent link="body_link"/>
     <child link="left_drive_wheel_link"/>
@@ -84,5 +84,5 @@
   </joint>
   <joint name="right_drive_wheel_joint" type="continuous">
-    <origin rpy="0 1.571 1.571" xyz="0 -0.158 -0.0599"/>
+    <origin rpy="0 1.571 1.571" xyz="0 -0.140 -0.0599"/>
     <parent link="body_link"/>
     <child link="right_drive_wheel_link"/>
@@ -93,5 +93,5 @@
   <!-- Caster wheels joint -->
   <joint name="front_caster_wheel_yaw_joint" type="continuous">
-    <origin rpy="0 0 0" xyz="0.158 0 -0.0775"/>
+    <origin rpy="0 0 0" xyz="0.140 0 -0.0775"/>
     <parent link="body_link"/>
     <child link="front_caster_wheel_yaw_link"/>
@@ -117,5 +117,5 @@
   </joint>
   <joint name="back_caster_wheel_yaw_joint" type="continuous">
-    <origin rpy="0 0 0" xyz="-0.158 0 -0.0775"/>
+    <origin rpy="0 0 0" xyz="-0.140 0 -0.0775"/>
     <parent link="body_link"/>
     <child link="back_caster_wheel_yaw_link"/>

Commit message: Update world

File: urdf/barista_robot_model.urdf (robot description, URDF)
Before this commit: robot barista_robot, 16 links, 15 joints
Links:
- added link laser_scanner_frame
- link laser_scanner_link: geometry collision cylinder length=0.0188 radius=0.0327; visual mesh filename=package://barista_robot_description/meshes/hokuyo_urg_04lx.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 scale=1 1 1
Joints:
- added joint laser_scanner_frame_joint: type fixed, parent laser_scanner_link, child laser_scanner_frame, origin xyz=0 0 0.06 rpy=0 0 0

File: xacro/barista_robot_model.urdf.xacro (robot description, xacro)
@@ -153,4 +153,9 @@
       <child link="laser_scanner_link"/>
     </joint>
+    <joint name="laser_scanner_frame_joint" type="fixed">
+      <origin rpy="0 0 0" xyz="0 0 0.06"/>
+      <parent link="laser_scanner_link"/>
+      <child link="laser_scanner_frame"/>
+    </joint>
   </xacro:if>
 </robot>

File: xacro/laser_scanner.xacro (robot description, xacro)
@@ -1,6 +1,6 @@
 <?xml version="1.0"?>
 <robot xmlns:xacro="http://www.ros.org/wiki/xacro">
-<!-- <xacro:property name="laser_scanner_radius" value="0.0327"/>
-<xacro:property name="laser_scanner_length" value="0.0188"/> -->
+<xacro:property name="laser_scanner_radius" value="0.0327"/>
+<xacro:property name="laser_scanner_length" value="0.0188"/>
 <xacro:macro name="laser_scanner">
   <link name="laser_scanner_link">
@@ -14,6 +14,6 @@
     <collision>
       <geometry>
-        <mesh filename="package://barista_robot_description/meshes/hokuyo_urg_04lx.dae" scale="1 1 1"/>
-        <!-- <cylinder radius="${laser_scanner_radius}" length="${laser_scanner_length}"/> -->
+        <!-- <mesh filename="package://barista_robot_description/meshes/hokuyo_urg_04lx.dae" scale="1 1 1"/> -->
+        <cylinder radius="${laser_scanner_radius}" length="${laser_scanner_length}"/>
       </geometry>
     </collision>
@@ -23,4 +23,6 @@
     </inertial>
   </link>
+  <link name="laser_scanner_frame">
+  </link>
 </xacro:macro>
 </robot>

File: xacro/model_plugins.xacro (robot description, xacro)
@@ -40,5 +40,5 @@
 </xacro:macro>
 <xacro:macro name="laser_scanner_plugin">
-  <gazebo reference="laser_scanner_link">
+  <gazebo reference="laser_scanner_frame">
     <sensor name="sensor_ray" type="ray">
         <pose>0 0 0 0 0 0</pose>
@@ -48,6 +48,6 @@
               <samples>200</samples>
               <resolution>1.0</resolution>
-              <min_angle>-3.14</min_angle>
-              <max_angle>3.14</max_angle>
+              <min_angle>-1.57</min_angle>
+              <max_angle>1.57</max_angle>
             </horizontal>
           </scan>
@@ -59,11 +59,11 @@
         <always_on>true</always_on>
         <visualize>true</visualize>
-        <update_rate>100.0</update_rate>
+        <update_rate>50.0</update_rate>
         <plugin name="laser" filename="libgazebo_ros_ray_sensor.so">
           <ros>
-            <namespace>/</namespace>
             <remapping>~/out:=scan</remapping>
           </ros>
           <output_type>sensor_msgs/LaserScan</output_type>
+          <frame_name>laser_scanner_frame</frame_name>
         </plugin>
       </sensor>
