Commit message: Update drive wheel name xacro

File: xacro/barista_robot_model.urdf.xacro (robot description, xacro)
@@ -11,6 +11,6 @@
 <xacro:include filename="$(find barista_robot_description)/xacro/standoff_rod.xacro" />
 <xacro:include filename="$(find barista_robot_description)/xacro/barista_robot_model.gazebo.xacro" />
-<xacro:drive_wheel drive_wheel_name="left_drive_wheel"/>
-<xacro:drive_wheel drive_wheel_name="right_drive_wheel"/>
+<xacro:drive_wheel drive_wheel_name="left_wheel"/>
+<xacro:drive_wheel drive_wheel_name="right_wheel"/>
 <xacro:caster_wheel caster_wheel_name="front_caster_wheel"/>
 <xacro:caster_wheel caster_wheel_name="back_caster_wheel"/>
@@ -75,16 +75,16 @@
   </joint>
   <!-- Wheels joint -->
-  <joint name="left_drive_wheel_joint" type="continuous">
+  <joint name="left_wheel_joint" type="continuous">
     <origin rpy="0 1.571 1.571" xyz="0 0.140 -0.0599"/>
     <parent link="body_link"/>
-    <child link="left_drive_wheel_link"/>
+    <child link="left_wheel_link"/>
     <axis rpy="0 0 0" xyz="0 0 1"/>
     <limit effort="10000" velocity="1000"/>
     <joint_properties damping="1.0" friction="1.0"/>
   </joint>
-  <joint name="right_drive_wheel_joint" type="continuous">
+  <joint name="right_wheel_joint" type="continuous">
     <origin rpy="0 1.571 1.571" xyz="0 -0.140 -0.0599"/>
     <parent link="body_link"/>
-    <child link="right_drive_wheel_link"/>
+    <child link="right_wheel_link"/>
     <axis rpy="0 0 0" xyz="0 0 1"/>
     <limit effort="10000" velocity="1000"/>

File: xacro/model_plugins.xacro (robot description, xacro)
@@ -8,6 +8,6 @@
       </ros>
       <update_rate>30.0</update_rate>
-      <joint_name>left_drive_wheel_joint</joint_name>
-      <joint_name>right_drive_wheel_joint</joint_name>
+      <joint_name>left_wheel_joint</joint_name>
+      <joint_name>right_wheel_joint</joint_name>
       <joint_name>front_caster_wheel_yaw_joint</joint_name>
       <joint_name>front_caster_wheel_roll_joint</joint_name>
@@ -23,6 +23,6 @@
     <plugin filename="libgazebo_ros_diff_drive.so" name="differential_drive_controller">
       <!-- wheels -->
-      <left_joint>left_drive_wheel_joint</left_joint>
-      <right_joint>right_drive_wheel_joint</right_joint>
+      <left_joint>left_wheel_joint</left_joint>
+      <right_joint>right_wheel_joint</right_joint>
       <!-- kinematics -->
       <wheel_separation>0.316</wheel_separation>
