Commit message: Checkpoint 8 - Part 1: simulation of multiple robots

File: xacro/barista_robot_model.gazebo.xacro (robot description, xacro)
@@ -8,4 +8,20 @@
     <material>Gazebo/Blue</material>
   </gazebo>
+  <xacro:if value="${robot_name == 'Morty'}">
+    <gazebo reference="body_link">
+      <material>Gazebo/Red</material>
+    </gazebo>
+    <gazebo reference="cup_holder_tray_link">
+      <material>Gazebo/Red</material>
+    </gazebo>
+  </xacro:if>
+  <xacro:if value="${robot_name == 'Rick'}">
+    <gazebo reference="body_link">
+      <material>Gazebo/Blue</material>
+    </gazebo>
+    <gazebo reference="cup_holder_tray_link">
+      <material>Gazebo/Blue</material>
+    </gazebo>
+  </xacro:if>
   <gazebo reference="standoff_rod_1_link">
     <material>Gazebo/White</material>

File: xacro/barista_robot_model.urdf.xacro (robot description, xacro)
@@ -1,4 +1,5 @@
 <?xml version="1.0"?>
 <robot xmlns:xacro="http://www.ros.org/wiki/xacro" name="barista_robot">
+<xacro:property name="robot_name" value="$(arg robot_name)"/>
 <xacro:property name="include_laser" value="$(arg include_laser)"/>
 <xacro:arg name="include_laser" default="true"/>
@@ -37,4 +38,10 @@
       </geometry>
       <material name="blue"/>
+      <xacro:if value="${robot_name == 'Rick'}">
+        <material name="blue"/>
+      </xacro:if>
+      <xacro:if value="${robot_name == 'Morty'}">
+        <material name="red"/>
+      </xacro:if>
     </visual>
     <collision>

File: xacro/cup_holder_tray.xacro (robot description, xacro)
@@ -10,4 +10,10 @@
       </geometry>
       <material name="blue"/>
+      <xacro:if value="${robot_name == 'Rick'}">
+        <material name="blue"/>
+      </xacro:if>
+      <xacro:if value="${robot_name == 'Morty'}">
+        <material name="red"/>
+      </xacro:if>
     </visual>
     <collision>

File: xacro/model_plugins.xacro (robot description, xacro)
@@ -5,4 +5,5 @@
     <plugin name="barista_robot_joint_state" filename="libgazebo_ros_joint_state_publisher.so">
       <ros>
+          <namespace>/${robot_name}</namespace>
           <remapping>~/out:=joint_states</remapping>
       </ros>
@@ -22,4 +23,8 @@
   <gazebo>
     <plugin filename="libgazebo_ros_diff_drive.so" name="differential_drive_controller">
+      <ros>
+        <namespace>/${robot_name}</namespace>
+        <remapping>/cmd_vel:=cmd_vel</remapping>
+      </ros>
       <!-- wheels -->
       <left_joint>left_wheel_joint</left_joint>
@@ -34,6 +39,6 @@
       <publish_odom>true</publish_odom>
       <publish_odom_tf>true</publish_odom_tf>
-      <odometry_frame>odom</odometry_frame>
-      <robot_base_frame>base_link</robot_base_frame>
+      <odometry_frame>${robot_name}/odom</odometry_frame>>
+      <robot_base_frame>${robot_name}/base_link</robot_base_frame>
     </plugin>
   </gazebo>
@@ -62,8 +67,9 @@
         <plugin name="laser" filename="libgazebo_ros_ray_sensor.so">
           <ros>
+            <namespace>/${robot_name}</namespace>
             <remapping>~/out:=scan</remapping>
           </ros>
           <output_type>sensor_msgs/LaserScan</output_type>
-          <frame_name>laser_scanner_frame</frame_name>
+          <frame_name>${robot_name}/laser_scanner_frame</frame_name>
         </plugin>
       </sensor>

Commit message: Update launch, urdf and xacro files for unity

File: xacro/barista_robot_model.gazebo.xacro (robot description, xacro)
@@ -2,10 +2,12 @@
 <robot xmlns:xacro="http://www.ros.org/wiki/xacro">
 <xacro:macro name="gazebo_elements">
-  <gazebo reference="body_link">
-    <material>Gazebo/Blue</material>
-  </gazebo>
-  <gazebo reference="cup_holder_tray_link">
-    <material>Gazebo/Blue</material>
-  </gazebo>
+  <xacro:if value="${robot_name == 'rick' or robot_name == 'barista_robot'}">
+    <gazebo reference="body_link">
+      <material>Gazebo/Blue</material>
+    </gazebo>
+    <gazebo reference="cup_holder_tray_link">
+      <material>Gazebo/Blue</material>
+    </gazebo>
+  </xacro:if>
   <xacro:if value="${robot_name == 'morty'}">
     <gazebo reference="body_link">
@@ -14,12 +16,4 @@
     <gazebo reference="cup_holder_tray_link">
       <material>Gazebo/Red</material>
-    </gazebo>
-  </xacro:if>
-  <xacro:if value="${robot_name == 'rick'}">
-    <gazebo reference="body_link">
-      <material>Gazebo/Blue</material>
-    </gazebo>
-    <gazebo reference="cup_holder_tray_link">
-      <material>Gazebo/Blue</material>
     </gazebo>
   </xacro:if>

File: xacro/barista_robot_model.urdf.xacro (robot description, xacro)
@@ -37,6 +37,5 @@
         <cylinder radius="0.178" length="0.155"/>
       </geometry>
-      <material name="blue"/>
-      <xacro:if value="${robot_name == 'rick'}">
+      <xacro:if value="${robot_name == 'rick' or robot_name == 'barista_robot'}">
         <material name="blue"/>
       </xacro:if>

File: xacro/cup_holder_tray.xacro (robot description, xacro)
@@ -9,6 +9,5 @@
         <cylinder radius="${cup_holder_tray_radius}" length="${cup_holder_tray_length}"/>
       </geometry>
-      <material name="blue"/>
-      <xacro:if value="${robot_name == 'rick'}">
+      <xacro:if value="${robot_name == 'rick' or robot_name == 'barista_robot'}">
         <material name="blue"/>
       </xacro:if>

File: xacro/model_plugins.xacro (robot description, xacro)
@@ -5,5 +5,7 @@
     <plugin name="barista_robot_joint_state" filename="libgazebo_ros_joint_state_publisher.so">
       <ros>
+        <xacro:if value="${robot_name == 'rick' or robot_name == 'morty'}">
           <namespace>/${robot_name}</namespace>
+        </xacro:if>
           <remapping>~/out:=joint_states</remapping>
       </ros>
@@ -24,5 +26,7 @@
     <plugin filename="libgazebo_ros_diff_drive.so" name="differential_drive_controller">
       <ros>
-        <namespace>/${robot_name}</namespace>
+        <xacro:if value="${robot_name == 'rick' or robot_name == 'morty'}">
+          <namespace>/${robot_name}</namespace>
+        </xacro:if>
         <remapping>/cmd_vel:=cmd_vel</remapping>
       </ros>
@@ -39,6 +43,12 @@
       <publish_odom>true</publish_odom>
       <publish_odom_tf>true</publish_odom_tf>
-      <odometry_frame>${robot_name}/odom</odometry_frame>>
-      <robot_base_frame>${robot_name}/base_link</robot_base_frame>
+      <xacro:if value="${robot_name == 'rick' or robot_name == 'morty'}">
+        <odometry_frame>${robot_name}/odom</odometry_frame>
+        <robot_base_frame>${robot_name}/base_link</robot_base_frame>
+      </xacro:if>
+      <xacro:if value="${robot_name == 'barista_robot'}">
+        <odometry_frame>odom</odometry_frame>
+        <robot_base_frame>base_link</robot_base_frame>
+      </xacro:if>
     </plugin>
   </gazebo>
@@ -67,9 +77,16 @@
         <plugin name="laser" filename="libgazebo_ros_ray_sensor.so">
           <ros>
-            <namespace>/${robot_name}</namespace>
+            <xacro:if value="${robot_name == 'rick' or robot_name == 'morty'}">
+              <namespace>/${robot_name}</namespace>
+            </xacro:if>
             <remapping>~/out:=scan</remapping>
           </ros>
           <output_type>sensor_msgs/LaserScan</output_type>
-          <frame_name>${robot_name}/laser_scanner_frame</frame_name>
+          <xacro:if value="${robot_name == 'rick' or robot_name == 'morty'}">
+            <frame_name>${robot_name}/laser_scanner_frame</frame_name>
+          </xacro:if>
+          <xacro:if value="${robot_name == 'barista_robot'}">
+            <frame_name>laser_scanner_frame</frame_name>
+          </xacro:if>
         </plugin>
       </sensor>
